Commit message: bolt definitions

File: urdf/bolt.urdf (robot description, URDF)
Before this commit: robot bolt, 9 links, 8 joints
Links:
- link FL_FOOT: geometry collision mesh filename=../meshes/stl/bolt_foot.stl; visual mesh filename=../meshes/stl/bolt_foot.stl
- link FL_LOWER_LEG: geometry collision mesh filename=../meshes/stl/lower_leg_200mm_left_side.stl; visual mesh filename=../meshes/stl/lower_leg_200mm_left_side.stl
- link FL_SHOULDER: geometry collision mesh filename=../meshes/stl/bolt_hip_fe_left_side.stl; visual mesh filename=../meshes/stl/bolt_hip_fe_left_side.stl
- link FL_UPPER_LEG: geometry collision mesh filename=../meshes/stl/upper_leg_200mm_left_side.stl; visual mesh filename=../meshes/stl/upper_leg_200mm_left_side.stl
- link FR_FOOT: geometry collision mesh filename=../meshes/stl/bolt_foot.stl; visual mesh filename=../meshes/stl/bolt_foot.stl
- link FR_LOWER_LEG: geometry collision mesh filename=../meshes/stl/lower_leg_200mm_right_side.stl; visual mesh filename=../meshes/stl/lower_leg_200mm_right_side.stl
- link FR_SHOULDER: geometry collision mesh filename=../meshes/stl/bolt_hip_fe_right_side.stl; visual mesh filename=../meshes/stl/bolt_hip_fe_right_side.stl
- link FR_UPPER_LEG: geometry collision mesh filename=../meshes/stl/upper_leg_200mm_right_side.stl; visual mesh filename=../meshes/stl/upper_leg_200mm_right_side.stl
- link base_link: geometry collision mesh filename=../meshes/stl/bolt_body.stl; visual mesh filename=../meshes/stl/bolt_body.stl

Commit message: ajout capsule urdf

File: urdf/bolt.urdf (robot description, URDF)
Before this commit: robot bolt, 9 links, 8 joints
Links:
- link FL_FOOT: mass 0.00000000 -> 0.012; geometry collision sphere radius=0.02; visual mesh filename=../meshes/stl/bolt_foot.stl
- link FL_LOWER_LEG: geometry collision capsule length=0.227 radius=0.0135; visual mesh filename=../meshes/stl/lower_leg_200mm_left_side.stl
- link FL_SHOULDER: geometry visual mesh filename=../meshes/stl/bolt_hip_fe_left_side.stl
- link FL_UPPER_LEG: geometry collision capsule length=0.237 radius=0.022; visual mesh filename=../meshes/stl/upper_leg_200mm_left_side.stl
- link FR_FOOT: mass 0.00000000 -> 0.012; geometry collision sphere radius=0.02; visual mesh filename=../meshes/stl/bolt_foot.stl
- link FR_LOWER_LEG: geometry collision capsule length=0.227 radius=0.0135; visual mesh filename=../meshes/stl/lower_leg_200mm_right_side.stl
- link FR_SHOULDER: geometry visual mesh filename=../meshes/stl/bolt_hip_fe_right_side.stl
- link FR_UPPER_LEG: geometry collision capsule length=0.237 radius=0.022; visual mesh filename=../meshes/stl/upper_leg_200mm_right_side.stl
- link base_link: geometry collision box size=0.155 0.164 0.095; visual mesh filename=../meshes/stl/bolt_body.stl
