Commit message: added mass to feet and added shoulder touch reset

File: IsaacGymEnvs/assets/urdf/bolt.urdf (robot description, URDF)
Before this commit: robot bolt, 9 links, 8 joints
Links:
- link FL_FOOT: mass 0.00000000 -> 0.012
- link FL_LOWER_LEG: geometry collision mesh filename=../meshes/stl/lower_leg_200mm_left_side.stl; visual mesh filename=../meshes/stl/lower_leg_200mm_left_baseside.stl
- link FR_FOOT: mass 0.00000000 -> 0.012

Commit message: latest run

File: IsaacGymEnvs/assets/urdf/bolt.urdf (robot description, URDF)
Before this commit: robot bolt, 9 links, 8 joints
Links:
- link FL_FOOT: mass 0.012 -> 0.00000000
- link FL_LOWER_LEG: geometry collision mesh filename=../meshes/stl/lower_leg_200mm_left_side.stl; visual mesh filename=../meshes/stl/lower_leg_200mm_left_side.stl
- link FR_FOOT: mass 0.012 -> 0.00000000
