Commit message: changed bolt's urdf hip angles and removed clereance reward

File: IsaacGymEnvs/assets/urdf/bolt_new.urdf (robot description, URDF)
Before this commit: robot bolt, 9 links, 8 joints
Joints:
- joint FL_HAA: limit lower=-10 upper=10 effort=1000 velocity=1000 -> lower=-5 upper=5 effort=1000 velocity=1000
- joint FR_HAA: limit lower=-10 upper=10 effort=1000 velocity=1000 -> lower=-5 upper=5 effort=1000 velocity=1000

Commit message: train: new urdf that doesnt cross its legs

File: IsaacGymEnvs/assets/urdf/bolt_new.urdf (robot description, URDF)
Before this commit: robot bolt, 9 links, 8 joints
Links:
- link FL_LOWER_LEG: geometry collision cylinder length=0.1 radius=0.015; visual mesh filename=../meshes/stl/lower_leg_200mm_left_side.stl
- link FL_UPPER_LEG: geometry collision cylinder length=0.110 radius=0.028; visual mesh filename=../meshes/stl/upper_leg_200mm_left_side.stl
- link FR_LOWER_LEG: geometry collision cylinder length=0.1 radius=0.015; visual mesh filename=../meshes/stl/lower_leg_200mm_right_side.stl
- link FR_UPPER_LEG: geometry collision cylinder length=0.110 radius=0.028; visual mesh filename=../meshes/stl/upper_leg_200mm_right_side.stl
Joints:
- joint FL_HAA: limit lower=-5 upper=5 effort=1000 velocity=1000 -> lower=-10 upper=10 effort=1000 velocity=1000
- joint FR_HAA: limit lower=-5 upper=5 effort=1000 velocity=1000 -> lower=-10 upper=10 effort=1000 velocity=1000
